Commit message: Изменены названия

File: src/armbot_description/urdf/armbot_description.urdf (robot description, URDF)
Before this commit: robot МР.300821.000.000 Манипулятор роботизированный.SLDASM, 7 links, 6 joints
Links:
- link base_link: geometry collision mesh filename=package://armbot_description/meshes/base_link.STL; visual mesh filename=package://armbot_description/meshes/base_link.STL
- link link_1: geometry collision mesh filename=package://armbot_description/meshes/link_1.STL; visual mesh filename=package://armbot_description/meshes/link_1.STL
- link link_2: geometry collision mesh filename=package://armbot_description/meshes/link_2.STL; visual mesh filename=package://armbot_description/meshes/link_2.STL
- link link_3: geometry collision mesh filename=package://armbot_description/meshes/link_3.STL; visual mesh filename=package://armbot_description/meshes/link_3.STL
- link link_4: geometry collision mesh filename=package://armbot_description/meshes/link_4.STL; visual mesh filename=package://armbot_description/meshes/link_4.STL
- link link_end: geometry collision mesh filename=package://armbot_description/meshes/link_end.STL; visual mesh filename=package://armbot_description/meshes/link_end.STL
- link link_grip: geometry collision mesh filename=package://armbot_description/meshes/link_grip.STL; visual mesh filename=package://armbot_description/meshes/link_grip.STL

Commit message: Обновлены файлы

File: src/armbot_description/urdf/armbot_description.urdf (robot description, URDF)
Before this commit: robot armbot_description, 7 links, 6 joints
Joints:
- joint joint_3: type fixed -> revolute
- joint joint_4: type fixed -> revolute

Commit message: Визуализация и симуляция

File: src/armbot_description/urdf/armbot_description.urdf (robot description, URDF)
Before this commit: robot armbot_description, 7 links, 6 joints
Joints:
- joint joint_3: origin xyz=0.11065 -0.077347 -0.011298 rpy=3.1416 0 -2.3727 -> xyz=0.13278 -0.024396 -0.011298 rpy=3.1416 0 -2.8607
- joint joint_4: origin xyz=0.16 0 -0.0068996 rpy=-3.1416 0 -0.80186 -> xyz=0.16 0 -0.0068996 rpy=-3.1416 0 -1.2899

File: src/armbot_description/urdf/model_best/armbot.gazebo.urdf (robot description, URDF)
Before this commit: robot armbot, 10 links, 9 joints
Links:
- link base_link: geometry collision mesh filename=package://armbot_description/meshes/model_best/base_link.STL; visual mesh filename=package://armbot_description/meshes/model_best/base_link.STL
- link link_1: geometry collision mesh filename=package://armbot_description/meshes/model_best/link_1.STL; visual mesh filename=package://armbot_description/meshes/model_best/link_1.STL
- link link_2: geometry collision mesh filename=package://armbot_description/meshes/model_best/link_2.STL; visual mesh filename=package://armbot_description/meshes/model_best/link_2.STL
- link link_3: geometry collision mesh filename=package://armbot_description/meshes/model_best/link_3.STL; visual mesh filename=package://armbot_description/meshes/model_best/link_3.STL
- link link_4: geometry collision mesh filename=package://armbot_description/meshes/model_best/link_4.STL; visual mesh filename=package://armbot_description/meshes/model_best/link_4.STL
- link link_end: geometry collision mesh filename=package://armbot_description/meshes/model_best/link_end.STL; visual mesh filename=package://armbot_description/meshes/model_best/link_end.STL
